Commit message: [Montessori] Sort with coraplex's own actions and measure the space under each hole
The robot no longer drives its own gripper. Picking a piece up is coraplex's
PickUpAction and putting it down is its PlaceAction, executed as giskard motion
statecharts under the simulated_robot execution environment, so a scripted run
commands the robot the way any other plan in this workspace does rather than solving
inverse kinematics of its own and setting joint positions by hand.

A simulation is built against one kinematic model and cannot follow a change to it,
and a grasp re-parents what it takes hold of, so SimulatedScene now builds its MuJoCo
mirror on demand and stop() drops it. A step that commands the robot lets go of the
simulation first; the next stretch of physics mirrors the world as it then is. The
scene's own physics is unchanged: gravity settles it, the pusher shoves a piece, and a
released piece falls through its hole.

The space under a hole is measured rather than stated. MontessoriWorld builds each
hole's landing region from the free space the hole's own footprint leaves down to the
table - a graph of convex sets over the board's and drawers' collision geometry - so
the region is the shaft that is actually open, and the hand-chosen margin and top
clearance are gone. A hole carries its own landing region, so a scene reads it off the
hole instead of spelling a name.

Two custom dataclass exceptions replace bare KeyErrors: NoSuchPieceError when a scene
is asked about a piece its layout never placed, and HoleHasNoLandingRegionError when a
hole was never measured under.

The test dataset's pincer gains a three-axis wrist, so a grasp can be oriented, and a
grasp frame between its finger tips, so an action that takes the tool frame to a piece
puts the fingers around it.

Made with the help of Claude.

Claude-Session: https://claude.ai/code/session_018F9bAELX9ep3v2wioNfCNB

File: test/experiments_test/dataset/synthetic_grasping_robot.urdf (robot description, URDF)
Before this commit: robot synthetic_grasping_robot, 9 links, 8 joints
Links:
- added link grasp_link, mass 0.01
- added link wrist_pitch_link, mass 0.2
- added link wrist_roll_link, mass 0.2
- added link wrist_yaw_link, mass 0.2
Joints:
- added joint grasp_joint: type fixed, parent pincer_link, child grasp_link, origin xyz=0 0 -0.03
- added joint wrist_pitch_joint: type revolute, parent wrist_roll_link, child wrist_pitch_link, axis 0 1 0, limit lower=-3.15 upper=3.15 effort=50 velocity=1
- added joint wrist_roll_joint: type revolute, parent lift_link, child wrist_roll_link, axis 1 0 0, limit lower=-3.15 upper=3.15 effort=50 velocity=1
- added joint wrist_yaw_joint: type revolute, parent wrist_pitch_link, child wrist_yaw_link, axis 0 0 1, limit lower=-3.15 upper=3.15 effort=50 velocity=1
- joint left_finger_joint: limit lower=0 upper=0.035 effort=50 velocity=1 -> lower=0 upper=0.05 effort=50 velocity=1
- joint pincer_joint: parent lift_link -> wrist_yaw_link
- joint right_finger_joint: limit lower=0 upper=0.035 effort=50 velocity=1 -> lower=0 upper=0.05 effort=50 velocity=1

Commit message: [Montessori] Film a scripted run, and tell a place how the piece is held
A scenario can now be filmed while it runs, with the repository's own
MuJoCo video recorder. A `SceneRecording` films the run and writes it as
one video, into `$MONTESSORI_SCENARIO_VIDEO_DIRECTORY` or a directory
beside whatever else the machine keeps temporarily.

A run is filmed in takes. A simulation is compiled against one kinematic
model and a grasp re-parents the piece, so no simulation carries a run
from end to end: `SimulatedScene` now lets go of what carries it whenever
the world's model changes, rather than each robot-commanding step
remembering to let go first, and a recording is cut and taken up again at
the same moments. The film is made from the simulation carrying the run
rather than from a second one beside it, so filming leaves the run doing
exactly what it did unfilmed -- measured to the last digit, and pinned by
a test.

What the film does not show is the carrying: while the robot holds the
piece, the world cannot be exported to MuJoCo at all, since the piece
keeps the free connection it stood on the table with and a free
connection has to be on a top-level body.

`PlaceAction` gains an optional `grasp_description`, so a place performed
in a plan of its own can be told how the object it is holding is held
rather than falling back to a grasp that did not happen. The sorting run
tells it, which turns the gripper to hold the piece from above rather
than from the front.

The mimic pincer carries visual geometry as well as collision, so the
hand is in the picture, and the experiments CI job exports MUJOCO_GL=egl,
which offscreen rendering needs before Python imports MuJoCo.

Made with the help of Claude.

Claude-Session: https://claude.ai/code/session_018F9bAELX9ep3v2wioNfCNB

File: test/experiments_test/dataset/synthetic_grasping_robot.urdf (robot description, URDF)
Before this commit: robot synthetic_grasping_robot, 13 links, 12 joints
Links:
- link left_fingertip_link: geometry collision box size=0.02 0.01 0.05; visual box size=0.02 0.01 0.05
- link pincer_link: geometry collision box size=0.04 0.08 0.02; visual box size=0.04 0.08 0.02
- link right_fingertip_link: geometry collision box size=0.02 0.01 0.05; visual box size=0.02 0.01 0.05
